File: openSTM32F4_LQFP64.sch (KiCad schematic (older format))
At the start: 77 parts, among them J1 Jack-DC, J10 Conn_01x04, J11 Conn_01x04, J12 Conn_01x05, J13 USB_B_Micro, J14 Conn_01x04, J15 Conn_01x04, J16 Conn_01x05, J17 Conn_01x06, J18 Conn_01x04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

Commit message: update jackDC mounting pin
Parts:
- removed J1: Jack-DC, Connector_BarrelJack:BarrelJack_Wuerth_6941xx301002, symbol Connector:Jack-DC
- added J1: Barrel_Jack_Switch, Connector_BarrelJack:BarrelJack_Wuerth_6941xx301002, symbol Connector:Barrel_Jack_Switch
- U6: footprint footprints:openstm_outline -> footprints:openSTM32F4_LQFP64_outline
Connections:
- wire segments 167 -> 168
Changed lines of the file:
@@
 	1550 6850 1800 6850
 Connection ~ 1800 6850
-$Comp
-L Connector:Jack-DC J1
-U 1 1 5EC5DDC2
-P 1000 6950
-F 0 "J1" H 1057 7275 50  0000 C CNN
-F 1 "Jack-DC" H 1057 7184 50  0000 C CNN
-F 2 "Connector_BarrelJack:BarrelJack_Wuerth_6941xx301002" H 1050 6910 50  0001 C CNN
-F 3 "~" H 1050 6910 50  0001 C CNN
-	1    1000 6950
-	1    0    0    -1
-$EndComp
 Wire Wire Line
 	1550 7150 1550 7450
@@
 F 0 "U6" H 7440 6896 50  0000 L CNN
 F 1 "outline" H 7440 6805 50  0000 L CNN
-F 2 "footprints:openstm_outline" H 7300 6850 50  0001 C CNN
+F 2 "footprints:openSTM32F4_LQFP64_outline" H 7300 6850 50  0001 C CNN
 F 3 "" H 7300 6850 50  0001 C CNN
 	1    7300 6850
@@
 Text Notes 9500 1800 0    118  ~ 24
 STLINK
+$Comp
+L Connector:Barrel_Jack_Switch J1
+U 1 1 5EA9F141
+P 1000 6950
+F 0 "J1" H 1057 7267 50  0000 C CNN
+F 1 "Barrel_Jack_Switch" H 1057 7176 50  0000 C CNN
+F 2 "Connector_BarrelJack:BarrelJack_Wuerth_6941xx301002" H 1050 6910 50  0001 C CNN
+F 3 "~" H 1050 6910 50  0001 C CNN
+	1    1000 6950
+	1    0    0    -1
+$EndComp
+Wire Wire Line
+	1300 7050 1300 6950
+Connection ~ 1300 7050
 $EndSCHEMATC
