File: openSTM32F4_LQFP64.sch (KiCad schematic (older format))
At the start: 77 parts, among them J1 Barrel_Jack_Switch, J10 Conn_01x04, J11 Conn_01x04, J12 Conn_01x05, J13 USB_B_Micro, J14 Conn_01x04, J15 Conn_01x04, J16 Conn_01x05, J17 Conn_01x06, J18 Conn_01x04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

Commit message: update mpu9250 footprint
Parts:
- U4: footprint Sensor_Motion:InvenSense_QFN-24_3x3mm_P0.4mm -> footprints:MPU9250
Changed lines of the file:
@@
 F 0 "U4" H 6000 5850 50  0000 C CNN
 F 1 "MPU-9250" H 6300 5850 50  0000 C CNN
-F 2 "Sensor_Motion:InvenSense_QFN-24_3x3mm_P0.4mm" H 5750 4100 50  0001 C CNN
+F 2 "footprints:MPU9250" H 5750 4100 50  0001 C CNN
 F 3 "https://store.invensense.com/datasheets/invensense/MPU9250REV1.0.pdf" H 5750 4950 50  0001 C CNN
 	1    5750 5100
